File: pcb/mobo/mobo.kicad_pcb (KiCad board)
At the start: 2 copper layers, 51.6 x 89 mm, 72 parts, among them J1 SWD_10, J2 PEEL_MOTOR, J3 DRIVE_MOTOR, J4 SW1, J5 SPRING_FINGERS, J6 SW2, J7 SW1, J8 USART1, J9 SWD_10, U1 STM32F031C6Tx, U2 STM32F031K6Ux, U4 AP1117-33, U5 MC34063AD, U6 MAX3078E, U7 DRV8837, U8 DRV8837, Y1 8MHz

Commit message: Power supply mangling
Parts:
- removed D6: 1N5819, Diode_SMD:D_SOD-123
- removed the G*** at (107.0, 61.5)
- removed the G*** at (147.1, 31.1)
- removed the G*** at (122.0, 79.1)
- removed the G*** at (107.7, 98.4)
- removed R13: 0.33R, Resistor_SMD:R_0805_2012Metric
- removed R6: 5.6k, Resistor_SMD:R_0805_2012Metric
- removed REF**: OSHW-Symbol_6.7x6mm_Mask, feeder:OSHW-Symbol_6.7x6mm_Mask
- removed U5: MC34063AD, Package_SO:SOIC-8_3.9x4.9mm_P1.27mm
- added C15: 2.2u, Capacitor_SMD:C_0805_2012Metric, F.Cu at (125.4, 43.5)
- added C21: 10u, Capacitor_SMD:C_0805_2012Metric, F.Cu at (121.2, 49.8)
- added H1: , Feeder:M3_Countersunk, F.Cu at (145.8, 35.8)
- added H2: , Feeder:M3_Countersunk, F.Cu at (145.8, 47.8)
- added H3: , Feeder:M3_Countersunk, F.Cu at (109.3, 88.3)
- added H4: , Feeder:M3_Countersunk, F.Cu at (109.3, 69.8)
- added H5: , Feeder:M3_Countersunk, F.Cu at (138.3, 83.8)
- added H6: , Feeder:M3_Countersunk, F.Cu at (147.3, 79.8)
- added H7: , Feeder:M3_Countersunk, F.Cu at (147.3, 70.8)
- added L2: 22u, Feeder:L_4018, F.Cu at (120.7, 44.5)
- added R10: 23.2k, Resistor_SMD:R_0805_2012Metric, F.Cu at (124.7, 51.8)
- added R11: 10K, Resistor_SMD:R_0805_2012Metric, F.Cu at (124.7, 49.8)
- added R8: 10K, Resistor_SMD:R_0805_2012Metric, F.Cu at (136.8, 49.8)
- added U3: LV3842X, Package_TO_SOT_SMD:SOT-23-6, F.Cu at (136.8, 46.8)
- C12: value 100uF -> 2.2u; footprint Capacitor_SMD:C_Elec_6.3x7.7 -> Capacitor_SMD:C_0805_2012Metric
- C13: value 10u -> 22u; footprint Capacitor_SMD:C_0805_2012Metric -> Capacitor_SMD:CP_Elec_5x5.3
- C14: value 470pF -> 100n
- C16: value 470uF -> 10u; footprint Capacitor_SMD:C_Elec_6.3x7.7 -> Capacitor_SMD:C_0805_2012Metric
- C6: value 15pF -> 15p
- C9: value 10u -> 100n
- L1: value 220uH -> 22u; footprint Inductor_SMD:L_6.3x6.3_H3 -> Feeder:L_4018
- R9: value 39k -> 90.9k
- U4: value AP1117-33 -> LV3842X; footprint Package_TO_SOT_SMD:SOT-223-3_TabPin2 -> Package_TO_SOT_SMD:SOT-23-6
- moved C13 20.6 mm to (135.5, 38.8), turned to 0 degrees
- moved R9 20.5 mm to (136.8, 51.8), turned to 180 degrees
- moved C9 11.0 mm to (133.2, 47.8), turned to 0 degrees
- moved C14 8.37 mm to (121.2, 47.8), turned to 0 degrees
- moved C12 7.11 mm to (137.5, 43.5), turned to 0 degrees
- moved L1 6.19 mm to (132.8, 44.5), turned to 180 degrees
- moved U4 3.78 mm to (124.7, 46.8)
- moved C16 2.39 mm to (133.2, 49.8), turned to 0 degrees
Connections:
- C13 pad 1: +3V3 -> +VDC
- C14 pad 1: GND -> Net-(U4-SW)
- C14 pad 2: Net-(C14-Pad2) -> Net-(U4-BOOT)
- C9 pad 1: +10V -> Net-(U3-SW)
- C9 pad 2: GND -> Net-(U3-BOOT)
- L1 pad 1: Net-(D6-Pad1) -> Net-(U3-SW)
- U4 pad 1: GND -> Net-(U4-BOOT)
- U4 pad 2: +3V3 -> GND
- U4 pad 3: +10V -> Net-(U4-FB)
Routing:
- net +3V3: track 269.4 -> 294.3 mm, vias 19 -> 16
- net GND: track 39.6 -> 64.3 mm, vias 110 -> 138
- net +10V: track 86.7 -> 75.1 mm
- net Net-(U3-FB): track 14.5 -> 3.88 mm, vias 2 -> 0
- net +VDC: track 29.8 -> 40.2 mm
- net Net-(D6-Pad1): track 10.0 -> 0.00 mm
- net Net-(R13-Pad2): track 9.45 -> 0.00 mm, vias 2 -> 0
- net Net-(C14-Pad2): track 8.59 -> 0.00 mm
- net Net-(U4-FB): track 0.00 -> 3.88 mm
- net Net-(U4-SW): track 0.00 -> 3.01 mm
- net Net-(U3-SW): track 0.00 -> 3.01 mm
- net Net-(U3-BOOT): track 0.00 -> 1.66 mm
- net Net-(U4-BOOT): track 0.00 -> 1.66 mm
Other:
- outline, holes or cut-outs redrawn
- board text removed: "LumenPnP Feeder REV12 <<hash>> Opulo Inc."
