File: pcb/mobo/mobo.kicad_sch (KiCad schematic)
At the start: 66 parts, among them J1 SWD_10, J2 PEEL_MOTOR, J3 DRIVE_MOTOR, J4 SW1, J5 SPRING_FINGERS, J6 SW2, J7 SW1, J8 USART1, J9 SWD_10, U1 STM32F031C6Tx, U2 STM32F031K6Ux, U4 AP1117-33, U5 MC34063AD, U6 MAX3078E, U7 DRV8837, U8 DRV8837, Y1 8MHz

Commit message: Power supply mangling
Parts:
- removed C12: 100uF, Capacitor_SMD:C_Elec_6.3x7.7, symbol Device:C_Polarized_Small
- removed C13: 10u, Capacitor_SMD:C_0805_2012Metric, symbol Device:C_Small
- removed C16: 470uF, Capacitor_SMD:C_Elec_6.3x7.7, symbol Device:C_Polarized_Small
- removed D6: 1N5819, Diode_SMD:D_SOD-123, symbol Diode:1N5819
- removed L1: 220uH, Inductor_SMD:L_6.3x6.3_H3, symbol pspice:INDUCTOR
- removed R13: 0.33R, Resistor_SMD:R_0805_2012Metric, symbol Device:R_Small
- removed R6: 5.6k, Resistor_SMD:R_0805_2012Metric, symbol Device:R_Small
- removed U4: AP1117-33, Package_TO_SOT_SMD:SOT-223-3_TabPin2, symbol Regulator_Linear:AP1117-33
- removed U5: MC34063AD, Package_SO:SOIC-8_3.9x4.9mm_P1.27mm, symbol Regulator_Switching:MC34063AD
- added C12, C15: 2.2u, Capacitor_SMD:C_0805_2012Metric, symbol Device:C
- added C13: 22u, Capacitor_SMD:CP_Elec_5x5.3, symbol Device:C_Polarized
- added C16, C21: 10u, Capacitor_SMD:C_0805_2012Metric, symbol Device:C
- added L1, L2: 22u, Feeder:L_4018, symbol Device:L
- added R10: 23.2k, Resistor_SMD:R_0805_2012Metric, symbol Device:R_Small
- added R11, R8: 10K, Resistor_SMD:R_0805_2012Metric, symbol Device:R_Small
- added U3, U4: LV3842X, Package_TO_SOT_SMD:SOT-23-6, symbol Feeder:LV3842X
- C1, C2: Mouser Part Number (none) -> 603-CC805JRNPO9BN150
- C10, C11, C8: Mouser Part Number (none) -> 187-CL21A475KPFNNNG
- C14: value 470pF -> 100n; Mouser Part Number (none) -> 791-0805B104K500CT
- C17, C18, C19, C20, C3, C4, C5, C7: Mouser Part Number (none) -> 791-0805B104K500CT
- C6: value 15pF -> 15p; Mouser Part Number (none) -> 603-CC805JRNPO9BN150
- C9: value 10u -> 100n; JLCPCB C15850 -> C49678; LCSC C17024 -> C476766; Mouser Part Number (none) -> 791-0805B104K500CT
- D1: now not fitted
- D2: Mouser Part Number (none) -> 576-SM712-02HTG
- D3: Mouser Part Number (none) -> 859-LTSTC19HE1WTRS1
- D9: Mouser Part Number (none) -> 863-MMSZ4684T1G
- FID1, FID2, FID3, J8, TP1, TP2, TP3, TP4, TP5, TP6, TP7, TP8: now left out of the parts list
- J1: now not fitted; now left out of the parts list
- J2: Mouser Part Number (none) -> 538-53261-0271
- J3: Mouser Part Number (none) -> 538-53261-0671
- J4, J6, J7: Mouser Part Number (none) -> 179-TS314635B260RASM
- J5: Mouser Part Number (none) -> 581-009155005541006
- J9: footprint Connector_PinHeader_1.27mm:PinHeader_2x05_P1.27mm_Vertical_SMD -> feeder:SWD-No-Paste; now not fitted; now left out of the parts list
- R1: Mouser Part Number (none) -> 708-RMCF0805FG1K00
- R14: Mouser Part Number (none) -> 667-ERJ-P06J221V
- R15, R16: Mouser Part Number (none) -> 660-RK73H2ATTDD20R0F
- R17, R4, R7: Mouser Part Number (none) -> 603-RE0805FRE0710KL
- R2, R3, R5: Mouser Part Number (none) -> 603-RC0805JR-10470RL
- R9: value 39k -> 90.9k; Mouser Part Number (none) -> 71-CRCW0805-90.9K-E3
- U1: Mouser Part Number (none) -> 511-STM32F031C6T6
- U2: footprint Package_DFN_QFN:QFN-32-1EP_5x5mm_P0.5mm_EP3.45x3.45mm -> feeder:QFN-32-No-Paste; now left out of the parts list
- U6: Mouser Part Number (none) -> 701-SP3078EEN-L/TR
- U7, U8: Mouser Part Number (none) -> 595-DRV8837CDSGR
- Y1: Mouser Part Number (none) -> 520-80833B2QCVYTR
Connections:
- net +10V: now also C16.1, L1.2; no longer C9.1
- net +3V3: now also C21.1, L2.2, R10.2
- net +VDC: now also C12.1, C13.1, C15.1, U3.4 (EN), U3.5 (VIN), U4.4 (EN), U4.5 (VIN)
- net GND: now also C12.2, C13.2, C15.2, C16.2, C21.2, R11.1, R8.1, U3.2 (GND), U4.2 (GND); no longer C14.1, C9.2
- net at R9.1: now also R8.2, U3.3 (FB)
- net at C14.2: now also U4.1 (BOOT)
- new net: C9.1, L1.1, U3.6 (SW)
- new net: C9.2, U3.1 (BOOT)
- new net: R10.1, R11.2, U4.3 (FB)
- new net: C14.1, L2.1, U4.6 (SW)
Other:
- moved on the sheet: TP1, TP2
